File: Laika/sheets/ProjectArchitecture.kicad_sch (KiCad schematic)
At the start: 0 parts

Commit message: Revert "GPS"
Other:
- sheet GPS ports: added none; removed {GPS_DATA}
- sheet SoC ports: added none; removed {GPS_DATA}
Changed lines of the file:
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@@
-		)
-	)
-	(bus
-		(pts
-			(xy 139.7 101.6) (xy 160.02 101.6)
-		)
-		(stroke
-			(width 0)
-			(type default)
 		)
 	)
@@
 			)
 		)
-		(pin "{GPS_DATA}" bidirectional
-			(at 160.02 101.6 180)
-			(effects
-				(font
-					(size 1.27 1.27)
-				)
-				(justify left)
-			)
-		)
 		(instances
 			(project "Laika"
@@
 			(effects
 				(font
-					(size 1.27 1.27)
-				)
-				(justify right)
-			)
-		)
-		(pin "{GPS_DATA}" bidirectional
-			(at 139.7 101.6 0)
-			(effects
-				(font
