File: Laika/sheets/sensors/IMU.kicad_sch (KiCad schematic)
At the start: 0 parts

Commit message: Created schematic for LSM6DSRX IMU
Parts:
- added C17, C18: 100n, symbol Device:C
- added U7: LSM6DSRX, Package_LGA:LGA-14_3x2.5mm_P0.5mm_LayoutBorder3x4y, symbol LaikaSensors:LSM6DSRX
Connections:
- new net +3V3: C17.1, C18.1, U7.5 (VDDIO), U7.8 (VDD)
- new net GND: C17.2, C18.2, U7.2 (SDX), U7.3 (SCX), U7.6 (GND), U7.7 (GND)
- new net IMU_CS: U7.12 (CS)
- new net IMU_INT: U7.4 (INT1)
- new net IMU_SCLK: U7.13 (SCL)
- new net IMU_SDI: U7.14 (SDA)
- new net IMU_SDO: U7.1 (SDO/SA0)
- no-connect marks 0 -> 1
Other:
- note added: "IMU"
